Commit message: Added wheel encoders

File: src/roomba_description/urdf/roomba.urdf.xacro (robot description, xacro)
@@ -5,9 +5,9 @@
   <xacro:property name="base_width" value="0.110"/>
   <xacro:property name="base_height" value="0.006"/>
-  <!-- Top chassis parameters (adjust these based on your actual robot) -->
-  <xacro:property name="top_length" value="0.193"/>
-  <xacro:property name="top_width" value="0.110"/>
-  <xacro:property name="top_height" value="0.006"/>
-  <xacro:property name="chassis_separation" value="0.04"/>  <!-- Distance between bottom and top chassis -->
+  <!-- Top chassis parameters -->
+  <xacro:property name="top_length" value="0.15"/>
+  <xacro:property name="top_width" value="0.10"/>
+  <xacro:property name="top_height" value="0.02"/>
+  <xacro:property name="chassis_separation" value="0.04"/>
   <xacro:property name="wheel_radius" value="0.03"/>
   <xacro:property name="wheel_thickness" value="0.02"/>
@@ -30,4 +30,7 @@
   <material name="white">
     <color rgba="1.0 1.0 1.0 1.0"/>
+  </material>
+  <material name="yellow">
+    <color rgba="1.0 1.0 0.0 1.0"/>
   </material>
   <!-- Base Link (Bottom Chassis - for wheels) -->
@@ -118,4 +121,37 @@
   <xacro:wheel name="rear_left" x="-0.0625" y="0.074" z="0.011"/>
   <xacro:wheel name="rear_right" x="-0.0625" y="-0.074" z="0.011"/>
+  <!-- Encoder Macro -->
+  <xacro:macro name="encoder" params="name x y z">
+    <link name="${name}_encoder">
+      <visual>
+        <origin xyz="0 0 0" rpy="0 0 0"/>
+        <geometry>
+          <cylinder radius="0.005" length="0.008"/>
+        </geometry>
+        <material name="yellow"/>
+      </visual>
+      <collision>
+        <origin xyz="0 0 0" rpy="0 0 0"/>
+        <geometry>
+          <cylinder radius="0.005" length="0.008"/>
+        </geometry>
+      </collision>
+      <inertial>
+        <origin xyz="0 0 0" rpy="0 0 0"/>
+        <mass value="0.005"/>
+        <inertia ixx="0.000001" ixy="0.0" ixz="0.0"
+                 iyy="0.000001" iyz="0.0"
+                 izz="0.000001"/>
+      </inertial>
+    </link>
+    <joint name="${name}_encoder_joint" type="fixed">
+      <parent link="base_link"/>
+      <child link="${name}_encoder"/>
+      <origin xyz="${x} ${y} ${z}" rpy="0 0 0"/>
+    </joint>
+  </xacro:macro>
+  <!-- Create Encoders (attached to base_link) -->
+  <xacro:encoder name="front_left" x="0.0825" y="0.028" z="0.011"/>
+  <xacro:encoder name="back_right" x="-0.0825" y="-0.028" z="0.011"/>
   <!-- IMU Link (mounted on top chassis) -->
   <link name="imu_link">
@@ -144,5 +180,4 @@
     <parent link="top_chassis"/>
     <child link="imu_link"/>
-    <!-- Adjust these coordinates relative to top_chassis -->
     <origin xyz="0.05 0.01 ${top_height/2 + 0.005}" rpy="0 0 0"/>
   </joint>
@@ -173,5 +208,4 @@
     <parent link="top_chassis"/>
     <child link="ultrasonic_link"/>
-    <!-- Adjust these coordinates relative to top_chassis -->
     <origin xyz="0.06 0.03 ${top_height/2 + 0.01}" rpy="0 0 0"/>
   </joint>
@@ -202,5 +236,4 @@
     <parent link="top_chassis"/>
     <child link="camera_link"/>
-    <!-- Adjust these coordinates relative to top_chassis -->
     <origin xyz="0.05 -0.01 ${top_height/2 + 0.005}" rpy="0 0 0"/>
   </joint>

Commit message: Successfully Implemented ROS Controls

File: src/roomba_description/urdf/roomba.urdf.xacro (robot description, xacro)
@@ -12,4 +12,6 @@
   <xacro:property name="wheel_radius" value="0.03"/>
   <xacro:property name="wheel_thickness" value="0.02"/>
+    <!-- Distance between controlled wheels (diagonal) -->
+  <xacro:property name="wheel_separation" value="0.148"/>
   <!-- Material Definitions -->
   <material name="blue">
@@ -85,40 +87,122 @@
     <origin xyz="0 0 ${chassis_separation}" rpy="0 0 0"/>
   </joint>
-  <!-- Wheel Macro -->
-  <xacro:macro name="wheel" params="name x y z">
-    <link name="${name}_wheel">
-      <visual>
-        <origin xyz="0 0 0" rpy="${pi/2} 0 0"/>
-        <geometry>
-          <cylinder radius="${wheel_radius}" length="${wheel_thickness}"/>
-        </geometry>
-        <material name="black"/>
-      </visual>
-      <collision>
-        <origin xyz="0 0 0" rpy="${pi/2} 0 0"/>
-        <geometry>
-          <cylinder radius="${wheel_radius}" length="${wheel_thickness}"/>
-        </geometry>
-      </collision>
-      <inertial>
-        <origin xyz="0 0 0" rpy="${pi/2} 0 0"/>
-        <mass value="0.1"/>
-        <inertia ixx="0.0005" ixy="0.0" ixz="0.0"
-                 iyy="0.0005" iyz="0.0"
-                 izz="0.0009"/>
-      </inertial>
-    </link>
-    <joint name="${name}_wheel_joint" type="continuous">
-      <parent link="base_link"/>
-      <child link="${name}_wheel"/>
-      <origin xyz="${x} ${y} ${z}" rpy="0 0 0"/>
-      <axis xyz="0 1 0"/>
-    </joint>
-  </xacro:macro>
-  <!-- Create All Four Wheels (attached to base_link) -->
-  <xacro:wheel name="front_left" x="0.0625" y="0.074" z="0.011"/>
-  <xacro:wheel name="front_right" x="0.0625" y="-0.074" z="0.011"/>
-  <xacro:wheel name="rear_left" x="-0.0625" y="0.074" z="0.011"/>
-  <xacro:wheel name="rear_right" x="-0.0625" y="-0.074" z="0.011"/>
+  <!-- ===== CONTROLLED WHEELS (for ros2_control) ===== -->
+  <!-- Front Left Wheel - LEFT MOTOR (controlled) -->
+  <link name="front_left_wheel">
+    <visual>
+      <origin xyz="0 0 0" rpy="${pi/2} 0 0"/>
+      <geometry>
+        <cylinder radius="${wheel_radius}" length="${wheel_thickness}"/>
+      </geometry>
+      <material name="red"/>  <!-- Red = controlled -->
+    </visual>
+    <collision>
+      <origin xyz="0 0 0" rpy="${pi/2} 0 0"/>
+      <geometry>
+        <cylinder radius="${wheel_radius}" length="${wheel_thickness}"/>
+      </geometry>
+    </collision>
+    <inertial>
+      <origin xyz="0 0 0" rpy="${pi/2} 0 0"/>
+      <mass value="0.1"/>
+      <inertia ixx="0.0005" ixy="0.0" ixz="0.0"
+               iyy="0.0005" iyz="0.0"
+               izz="0.0009"/>
+    </inertial>
+  </link>
+  <joint name="front_left_wheel_joint" type="continuous">
+    <parent link="base_link"/>
+    <child link="front_left_wheel"/>
+    <origin xyz="0.0625 0.074 0.011" rpy="0 0 0"/>
+    <axis xyz="0 1 0"/>
+  </joint>
+  <!-- Rear Right Wheel - RIGHT MOTOR (controlled) -->
+  <link name="rear_right_wheel">
+    <visual>
+      <origin xyz="0 0 0" rpy="${pi/2} 0 0"/>
+      <geometry>
+        <cylinder radius="${wheel_radius}" length="${wheel_thickness}"/>
+      </geometry>
+      <material name="red"/>  <!-- Red = controlled -->
+    </visual>
+    <collision>
+      <origin xyz="0 0 0" rpy="${pi/2} 0 0"/>
+      <geometry>
+        <cylinder radius="${wheel_radius}" length="${wheel_thickness}"/>
+      </geometry>
+    </collision>
+    <inertial>
+      <origin xyz="0 0 0" rpy="${pi/2} 0 0"/>
+      <mass value="0.1"/>
+      <inertia ixx="0.0005" ixy="0.0" ixz="0.0"
+               iyy="0.0005" iyz="0.0"
+               izz="0.0009"/>
+    </inertial>
+  </link>
+  <joint name="rear_right_wheel_joint" type="continuous">
+    <parent link="base_link"/>
+    <child link="rear_right_wheel"/>
+    <origin xyz="-0.0625 -0.074 0.011" rpy="0 0 0"/>
+    <axis xyz="0 1 0"/>
+  </joint>
+  <!-- ===== PASSIVE WHEELS (for visualization only) ===== -->
+  <!-- Front Right Wheel - PASSIVE -->
+  <link name="front_right_wheel">
+    <visual>
+      <origin xyz="0 0 0" rpy="${pi/2} 0 0"/>
+      <geometry>
+        <cylinder radius="${wheel_radius}" length="${wheel_thickness}"/>
+      </geometry>
+      <material name="black"/>  <!-- Black = passive -->
+    </visual>
+    <collision>
+      <origin xyz="0 0 0" rpy="${pi/2} 0 0"/>
+      <geometry>
+        <cylinder radius="${wheel_radius}" length="${wheel_thickness}"/>
+      </geometry>
+    </collision>
+    <inertial>
+      <origin xyz="0 0 0" rpy="${pi/2} 0 0"/>
+      <mass value="0.1"/>
+      <inertia ixx="0.0005" ixy="0.0" ixz="0.0"
+               iyy="0.0005" iyz="0.0"
+               izz="0.0009"/>
+    </inertial>
+  </link>
+  <joint name="front_right_wheel_joint" type="continuous">
+    <parent link="base_link"/>
+    <child link="front_right_wheel"/>
+    <origin xyz="0.0625 -0.074 0.011" rpy="0 0 0"/>
+    <axis xyz="0 1 0"/>
+  </joint>
+  <!-- Rear Left Wheel - PASSIVE -->
+  <link name="rear_left_wheel">
+    <visual>
+      <origin xyz="0 0 0" rpy="${pi/2} 0 0"/>
+      <geometry>
+        <cylinder radius="${wheel_radius}" length="${wheel_thickness}"/>
+      </geometry>
+      <material name="black"/>  <!-- Black = passive -->
+    </visual>
+    <collision>
+      <origin xyz="0 0 0" rpy="${pi/2} 0 0"/>
+      <geometry>
+        <cylinder radius="${wheel_radius}" length="${wheel_thickness}"/>
+      </geometry>
+    </collision>
+    <inertial>
+      <origin xyz="0 0 0" rpy="${pi/2} 0 0"/>
+      <mass value="0.1"/>
+      <inertia ixx="0.0005" ixy="0.0" ixz="0.0"
+               iyy="0.0005" iyz="0.0"
+               izz="0.0009"/>
+    </inertial>
+  </link>
+  <joint name="rear_left_wheel_joint" type="continuous">
+    <parent link="base_link"/>
+    <child link="rear_left_wheel"/>
+    <origin xyz="-0.0625 0.074 0.011" rpy="0 0 0"/>
+    <axis xyz="0 1 0"/>
+  </joint>
   <!-- Encoder Macro -->
   <xacro:macro name="encoder" params="name x y z">
@@ -238,3 +322,30 @@
     <origin xyz="0.05 -0.01 ${top_height/2 + 0.005}" rpy="0 0 0"/>
   </joint>
+  <!-- ros2_control configuration - Uses the 2 controlled wheels -->
+  <ros2_control name="roomba_control" type="system">
+    <hardware>
+      <plugin>roomba_hardware/RoombaHardwareInterface</plugin>
+      <param name="wheel_radius">${wheel_radius}</param>
+      <param name="wheel_separation">${wheel_separation}</param>
+    </hardware>
+    <!-- Front Left = Left Motor -->
+    <joint name="front_left_wheel_joint">
+      <command_interface name="velocity">
+        <param name="min">-10.0</param>
+        <param name="max">10.0</param>
+      </command_interface>
+      <state_interface name="position"/>
+      <state_interface name="velocity"/>
+    </joint>
+    <!-- Rear Right = Right Motor -->
+    <joint name="rear_right_wheel_joint">
+      <command_interface name="velocity">
+        <param name="min">-10.0</param>
+        <param name="max">10.0</param>
+      </command_interface>
+      <state_interface name="position"/>
+      <state_interface name="velocity"/>
+    </joint>
+    <!-- front_right_wheel_joint and rear_left_wheel_joint are NOT controlled -->
+  </ros2_control>
 </robot>

Commit message: latest_changes

File: src/roomba_description/urdf/roomba.urdf.xacro (robot description, xacro)
@@ -146,6 +146,4 @@
     <axis xyz="0 1 0"/>
   </joint>
-  <!-- ===== PASSIVE WHEELS (for visualization only) ===== -->
-  <!-- Front Right Wheel - PASSIVE -->
   <link name="front_right_wheel">
     <visual>
@@ -154,5 +152,5 @@
         <cylinder radius="${wheel_radius}" length="${wheel_thickness}"/>
       </geometry>
-      <material name="black"/>  <!-- Black = passive -->
+      <material name="black"/>
     </visual>
     <collision>
@@ -176,5 +174,4 @@
     <axis xyz="0 1 0"/>
   </joint>
-  <!-- Rear Left Wheel - PASSIVE -->
   <link name="rear_left_wheel">
     <visual>
@@ -183,5 +180,5 @@
         <cylinder radius="${wheel_radius}" length="${wheel_thickness}"/>
       </geometry>
-      <material name="black"/>  <!-- Black = passive -->
+      <material name="black"/>
     </visual>
     <collision>
@@ -322,4 +319,32 @@
     <origin xyz="0.05 -0.01 ${top_height/2 + 0.005}" rpy="0 0 0"/>
   </joint>
+  <!-- LIDAR JOINT  -->
+  <link name="laser" >
+  <visual>
+  <origin xyz="0 0 0" rpy="0 0 0" />
+  <geometry>
+    <box size="0.045 0.045 0.035"/>
+  </geometry>
+  <material name="black"/>
+  </visual>
+  <collision>
+  <origin xyz="0 0 0" rpy="0 0 0" />
+  <geometry>
+    <box size="0.045 0.045 0.035"/>
+  </geometry>
+  </collision>
+  <inertial>
+    <origin xyz="0 0 0" rpy="0 0 0"/>
+    <mass value="0.01"/>
+    <inertia ixx="0.00001" ixy="0.0" ixz="0.0"
+              iyy="0.00001" iyz="0.0"
+              izz="0.00001"/>
+  </inertial>
+  </link>
+  <joint name="laser_joint" type="fixed">
+    <parent link="top_chassis" />
+    <child link="laser" />
+    <origin xyz="0 0 ${top_height/2 + 0.05}" rpy="0 0 0"/>
+  </joint>
   <!-- ros2_control configuration - Uses the 2 controlled wheels -->
   <ros2_control name="roomba_control" type="system">

Commit message: urdf change

File: src/roomba_description/urdf/roomba.urdf.xacro (robot description, xacro)
@@ -345,29 +345,5 @@
     <parent link="top_chassis" />
     <child link="laser" />
-    <origin xyz="0 0 ${top_height/2 + 0.05}" rpy="0 0 0"/>
-  </joint>
-  <!-- ros2_control configuration - Uses the 2 controlled wheels -->
-  <!-- <ros2_control name="roomba_control" type="system">
-    <hardware>
-      <plugin>roomba_hardware/RoombaHardwareInterface</plugin>
-      <param name="wheel_radius">${wheel_radius}</param>
-      <param name="wheel_separation">${wheel_separation}</param>
-    </hardware>
-    <joint name="front_left_wheel_joint">
-      <command_interface name="velocity">
-        <param name="min">-7.0</param>
-        <param name="max">7.0</param>
-      </command_interface>
-      <state_interface name="position"/>
-      <state_interface name="velocity"/>
-    </joint>
-    <joint name="rear_right_wheel_joint">
-      <command_interface name="velocity">
-        <param name="min">-7.0</param>
-        <param name="max">7.0</param>
-      </command_interface>
-      <state_interface name="position"/>
-      <state_interface name="velocity"/>
-    </joint>
-  </ros2_control> -->
+    <origin xyz="0 0 ${top_height/2 + 0.05}" rpy="0 0 3.145"/>
+  </joint>
 </robot>
